File: keyboard.kicad_sch (KiCad schematic)
At the start: 0 parts

Commit message: made electronic schema
Parts:
- added C? (x4): 0.1u, symbol Device:C_Small
- added C?: 1uF, symbol Device:C_Small
- added C? (x2): 22p, symbol Device:C_Small
- added C?: 10u, symbol Device:C_Small
- added D?: PRTR5V0U2X, Package_TO_SOT_SMD:SOT-143, symbol Power_Protection:PRTR5V0U2X
- added F?: 500m, symbol Device:Polyfuse_Small
- added J?: AVR-ISP-6, symbol Connector:AVR-ISP-6
- added R? (x2): 5.1k, symbol Device:R_Small
- added R? (x2): 10K, symbol Device:R_Small
- added R? (x2): 22, symbol Device:R_Small
- added U?: ATmega32U4-A, Package_QFP:TQFP-44_10x10mm_P0.8mm, symbol MCU_Microchip_ATmega:ATmega32U4-A
- added U?: ~, symbol usb:SW_SKQG
- added USB?: HRO-TYPE-C-31-M-12, symbol Type-C:HRO-TYPE-C-31-M-12
- added Y?: Crystal_GND24_Small, symbol Device:Crystal_GND24_Small
Connections:
- new net: R?.1, USB?.10 (CC2)
- new net: R?.2, U?.31 (PC6)
- new net: D?.2 (I/O1), R?.1, USB?.6 (DP1), USB?.8 (DP2)
- new net: R?.1, USB?.4 (CC1)
- new net: C?.1, U?.6 (UCAP)
- new net: D?.3 (I/O2), R?.1, USB?.5 (DN2), USB?.7 (DN1)
- new net +5V: C?.1, C?.1, C?.1, C?.1, C?.1, F?.2, J?.2 (VCC), R?.2, U?.14 (VCC), U?.2 (UVCC), U?.24 (AVCC), U?.34 (VCC), U?.44 (AVCC)
- new net D+: R?.2, U?.4 (D+)
- new net D-: R?.2, U?.3 (D-)
- new net GND: C?.2, C?.2, C?.2, C?.2, C?.2, C?.2, C?.2, D?.1 (GND), J?.6 (GND), R?.1, R?.2, R?.2, U?. (2), U?.15 (GND), U?.23 (GND), U?.35 (GND), U?.43 (GND), U?.5 (UGND), USB?.1 (GND), USB?.12 (GND), USB?.13 (SHIELD), Y?.2, Y?.4
- new net MISO: J?.1 (MISO), U?.11 (PB3)
- new net MOSI: J?.4 (MOSI), U?.10 (PB2)
- new net RESET: J?.5 (~{RST}), R?.1, U?. (2), U?.13 (~{RESET})
- new net SCK: J?.3 (SCK), U?.9 (PB1)
- new net VCC: D?.4 (VCC), F?.1, USB?.11 (VBUS), USB?.2 (VBUS)
- new net XTAL1: C?.1, U?.17 (XTAL1), Y?.1
- new net XTAL2: C?.1, U?.16 (XTAL2), Y?.3
- no-connect marks 0 -> 5

Commit message: started matrix
Other:
- added sheet matrix (matrix.kicad_sch)
Changed lines of the file:
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@@
+		)
+	)
+	(sheet
+		(at 58.42 158.75)
+		(size 12.7 3.81)
+		(exclude_from_sim no)
+		(in_bom yes)
+		(on_board yes)
+		(dnp no)
+		(fields_autoplaced yes)
+		(stroke
+			(width 0.1524)
+			(type solid)
+		)
+		(fill
+			(color 0 0 0 0.0000)
+		)
+		(property "Sheetname" "matrix"
+			(at 58.42 158.0384 0)
+			(effects
+				(font
+					(size 1.27 1.27)
+				)
+				(justify left bottom)
+			)
+		)
+		(property "Sheetfile" "matrix.kicad_sch"
+			(at 58.42 163.1446 0)
+			(effects
+				(font
+					(size 1.27 1.27)
+				)
+				(justify left top)
+			)
+		)
+		(instances
+			(project "keyboard"
+				(path "/e6cb590d-871d-49ba-8de3-d49ab73cdab4"
+					(page "2")
+				)
+			)
 		)
 	)
